File: _autosave-AmstradCPC6128PSU.kicad_pcb (KiCad board)
At the start: 2 copper layers, 35.6 x 22.9 mm, 3 parts, among them J1 DC 5V, J2 Mini-DIN-6, J3 DC 12V

Commit message: hmmm
Parts:
- moved J1 5.08 mm to (152.4, 85.1), turned to 270 degrees
Connections:
- J1 pad 1: Net-(J1-Pad1) -> /GND
- J1 pad 2: Net-(J1-Pad2) -> /+5V
- J2 pad 1: Net-(J2-Pad1) -> /+12V
- J2 pad 2: Net-(J2-Pad2) -> /+12V
- J2 pad 3: Net-(J1-Pad1) -> /+5V
- J2 pad 4: Net-(J2-Pad4) -> /GND
- J2 pad 5: Net-(J2-Pad5) -> /+5V
- J2 pad 6: Net-(J1-Pad2) -> /GND
- J3 pad 1: Net-(J2-Pad1) -> Net-(J3-Pad1)
- J3 pad 2: Net-(J2-Pad5) -> Net-(J3-Pad2)
Routing:
- net Net-(J1-Pad1): track 25.8 -> 0.00 mm
- net /+5V: track 0.00 -> 23.0 mm
- net Net-(J1-Pad2): track 22.3 -> 0.00 mm
- net Net-(J2-Pad1): track 18.6 -> 0.00 mm
- net Net-(J2-Pad5): track 17.1 -> 0.00 mm
Other:
- net class 5-12V 2A added: clearance 0.6, trace_width 0.8, via_dia 0.8, via_drill 0.4
Changed lines of the file:
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@@
     (thickness 1.6)
     (drawings 4)
-    (tracks 16)
+    (tracks 2)
     (zones 0)
     (modules 3)
-    (nets 7)
+    (nets 6)
   )
   (page A4)
@@
   )
   (net 0 "")
-  (net 1 "Net-(J1-Pad1)")
-  (net 2 "Net-(J1-Pad2)")
-  (net 3 "Net-(J2-Pad1)")
-  (net 4 "Net-(J2-Pad2)")
-  (net 5 "Net-(J2-Pad5)")
-  (net 6 "Net-(J2-Pad4)")
+  (net 1 /+5V)
+  (net 2 /GND)
+  (net 3 /+12V)
+  (net 4 "Net-(J3-Pad2)")
+  (net 5 "Net-(J3-Pad1)")
   (net_class Default "Ceci est la Netclass par défaut."
     (clearance 0.2)
@@
     (uvia_dia 0.3)
     (uvia_drill 0.1)
-    (add_net "Net-(J1-Pad1)")
-    (add_net "Net-(J1-Pad2)")
-    (add_net "Net-(J2-Pad1)")
-    (add_net "Net-(J2-Pad2)")
-    (add_net "Net-(J2-Pad4)")
-    (add_net "Net-(J2-Pad5)")
+    (add_net /GND)
+    (add_net "Net-(J3-Pad1)")
+    (add_net "Net-(J3-Pad2)")
+  )
+  (net_class "5-12V 2A" ""
+    (clearance 0.6)
+    (trace_width 0.8)
+    (via_dia 0.8)
+    (via_drill 0.4)
+    (uvia_dia 0.3)
+    (uvia_drill 0.1)
+    (add_net /+12V)
+    (add_net /+5V)
   )
   (module TerminalBlock:TerminalBlock_bornier-2_P5.08mm (layer F.Cu)
-    (at 152.4 90.17 90)
+    (at 152.4 85.09 270)
     (descr "simple 2-pin terminal block, pitch 5.08mm, revamped version of bornier2")
     (tags "terminal block bornier2")
-    (fp_text reference J1 (at 2.54 -5.08 90) (layer F.SilkS)
-      (effects (font (size 1 1) (thickness 0.15)))
-    )
-    (fp_text value "DC 5V" (at 2.54 5.08 90) (layer F.Fab)
+    (fp_text reference J1 (at 2.54 -5.08 270) (layer F.SilkS)
+      (effects (font (size 1 1) (thickness 0.15)))
+    )
+    (fp_text value "DC 5V" (at 2.54 5.08 270) (layer F.Fab)
       (effects (font (size 1 1) (thickness 0.15)))
     )
@@
     (fp_line (start -2.46 -3.75) (end -2.46 3.75) (layer F.Fab) (width 0.1))
     (fp_line (start -2.41 2.55) (end 7.49 2.55) (layer F.Fab) (width 0.1))
-    (fp_text user %R (at 2.54 0 90) (layer F.Fab)
-      (effects (font (size 1 1) (thickness 0.15)))
-    )
-    (pad 2 thru_hole circle (at 5.08 0 90) (size 3 3) (drill 1.52) (layers *.Cu *.Mask)
-      (net 2 "Net-(J1-Pad2)"))
-    (pad 1 thru_hole rect (at 0 0 90) (size 3 3) (drill 1.52) (layers *.Cu *.Mask)
-      (net 1 "Net-(J1-Pad1)"))
+    (fp_text user %R (at 2.54 0 270) (layer F.Fab)
+      (effects (font (size 1 1) (thickness 0.15)))
+    )
+    (pad 2 thru_hole circle (at 5.08 0 270) (size 3 3) (drill 1.52) (layers *.Cu *.Mask)
+      (net 1 /+5V))
+    (pad 1 thru_hole rect (at 0 0 270) (size 3 3) (drill 1.52) (layers *.Cu *.Mask)
+      (net 2 /GND))
     (model ${KISYS3DMOD}/TerminalBlock.3dshapes/TerminalBlock_bornier-2_P5.08mm.wrl
       (offset (xyz 2.539999961853027 0 0))
@@
     (pad 7 thru_hole oval (at -1.3 3.65 270) (size 4 2) (drill oval 3 1) (layers *.Cu *.Mask))
     (pad 6 thru_hole circle (at -4.7 -2.8 270) (size 1.6 1.6) (drill 0.8) (layers *.Cu *.Mask)
-      (net 2 "Net-(J1-Pad2)"))
+      (net 2 /GND))
     (pad 5 thru_hole circle (at 2.1 -2.8 270) (size 1.6 1.6) (drill 0.8) (layers *.Cu *.Mask)
-      (net 5 "Net-(J2-Pad5)"))
+      (net 1 /+5V))
     (pad 4 thru_hole circle (at -4.7 0 270) (size 1.6 1.6) (drill 0.8) (layers *.Cu *.Mask)
-      (net 6 "Net-(J2-Pad4)"))
+      (net 2 /GND))
     (pad 3 thru_hole circle (at 2.1 0 270) (size 1.6 1.6) (drill 0.8) (layers *.Cu *.Mask)
-      (net 1 "Net-(J1-Pad1)"))
+      (net 1 /+5V))
     (pad 2 thru_hole circle (at -2.6 0 270) (size 1.6 1.6) (drill 0.8) (layers *.Cu *.Mask)
-      (net 4 "Net-(J2-Pad2)"))
+      (net 3 /+12V))
     (pad 1 thru_hole rect (at 0 0 270) (size 1.6 1.6) (drill 0.8) (layers *.Cu *.Mask)
-      (net 3 "Net-(J2-Pad1)"))
+      (net 3 /+12V))
     (pad 7 thru_hole oval (at 5.55 2.85 270) (size 2 3.5) (drill oval 1 2.5) (layers *.Cu *.Mask))
     (pad 7 thru_hole oval (at -8.15 2.85 270) (size 2 3.5) (drill oval 1 2.5) (layers *.Cu *.Mask))
@@
     (pad 3 thru_hole roundrect (at -3 4.7 180) (size 3.5 3.5) (drill oval 3 1) (layers *.Cu *.Mask) (roundrect_rratio 0.25))
     (pad 2 thru_hole roundrect (at -6 0 180) (size 3 3.5) (drill oval 1 3) (layers *.Cu *.Mask) (roundrect_rratio 0.25)
-      (net 5 "Net-(J2-Pad5)"))
+      (net 4 "Net-(J3-Pad2)"))
     (pad 1 thru_hole rect (at 0 0 180) (size 3.5 3.5) (drill oval 1 3) (layers *.Cu *.Mask)
-      (net 3 "Net-(J2-Pad1)"))
+      (net 5 "Net-(J3-Pad1)"))
     (model ${KISYS3DMOD}/Connector_BarrelJack.3dshapes/BarrelJack_Horizontal.wrl
       (at (xyz 0 0 0))
@@
   (gr_line (start 156.21 105.41) (end 156.21 82.55) (layer Edge.Cuts) (width 0.15))
   (gr_line (start 120.65 105.41) (end 156.21 105.41) (layer Edge.Cuts) (width 0.15))
-  (segment (start 129.54 97.35) (end 135.45 91.44) (width 0.25) (layer F.Cu) (net 1))
-  (segment (start 150.65 90.17) (end 152.4 90.17) (width 0.25) (layer F.Cu) (net 1))
-  (segment (start 149.38 91.44) (end 150.65 90.17) (width 0.25) (layer F.Cu) (net 1))
-  (segment (start 135.45 91.44) (end 149.38 91.44) (width 0.25) (layer F.Cu) (net 1))
-  (segment (start 146.94 90.55) (end 152.4 85.09) (width 0.25) (layer F.Cu) (net 2))
-  (segment (start 132.34 90.55) (end 146.94 90.55) (width 0.25) (layer F.Cu) (net 2))
-  (segment (start 140.24 100.33) (end 142.24 100.33) (width 0.25) (layer F.Cu) (net 3))
-  (segment (start 130.854998 100.33) (end 140.24 100.33) (width 0.25) (layer F.Cu) (net 3))
-  (segment (start 128.414999 97.890001) (end 130.854998 100.33) (width 0.25) (layer F.Cu) (net 3))
-  (segment (start 128.414999 95.325001) (end 128.414999 97.890001) (width 0.25) (layer F.Cu) (net 3))
-  (segment (start 128.49 95.25) (end 128.414999 95.325001) (width 0.25) (layer F.Cu) (net 3))
-  (segment (start 129.54 95.25) (end 128.49 95.25) (width 0.25) (layer F.Cu) (net 3))
-  (segment (start 146.779545 98.869545) (end 148.24 100.33) (width 0.25) (layer F.Cu) (net 5))
-  (segment (start 146.059999 98.149999) (end 146.779545 98.869545) (width 0.25) (layer F.Cu) (net 5))
-  (segment (start 133.139999 98.149999) (end 146.059999 98.149999) (width 0.25) (layer F.Cu) (net 5))
-  (segment (start 132.34 97.35) (end 133.139999 98.149999) (width 0.25) (layer F.Cu) (net 5))
+  (segment (start 132.34 97.35) (end 139.52 90.17) (width 0.8) (layer F.Cu) (net 1))
+  (segment (start 139.52 90.17) (end 152.4 90.17) (width 0.8) (layer F.Cu) (net 1))
 )
