File: AmstradCPC6128PSU.sch (KiCad schematic (older format))
At the start: 3 parts, among them J1 DC 5V, J2 Mini-DIN-6, J3 DC 12V

Commit message: getting there
Parts:
- added H1, H2: MountingHole_Pad, MountingHole:MountingHole_2.2mm_M2_Pad_Via, symbol Mechanical:MountingHole_Pad
- added J4: Conn_01x04_Male, Connector_PinHeader_2.54mm:PinHeader_1x04_P2.54mm_Vertical, symbol Connector:Conn_01x04_Male
- J2: symbol Connector:Mini-DIN-6 -> custom_symbols:Mini-DIN_6pins
- J3: symbol Connector:Jack-DC -> Connector:Barrel_Jack_Switch
Connections:
- net +12V: now reaches J2.1, J3.1
- net +12V: now also J2.2, J4.1 (Pin_1)
- net +5V: now reaches J1.1 (Pin_1), J2.3
- net +5V: now also J2.5, J4.4 (Pin_4)
- net GND: now reaches J2.4
- net GND: now also J1.2 (Pin_2), J2.6, J2.7 (Shell), J3.2, H1.1, H2.1, J4.3 (Pin_3)
- new net SW: J3.3, J4.2 (Pin_2)
Changed lines of the file:
@@
 $EndDescr
 $Comp
-L Connector:Mini-DIN-6 J2
+L custom_symbols:Mini-DIN_6pins J2
 U 1 1 5EBB01DA
-P 3800 3350
-F 0 "J2" H 3800 3717 50  0000 C CNN
-F 1 "Mini-DIN-6" H 3800 3626 50  0000 C CNN
-F 2 "Custom_Footprints:Connector_Mini-DIN_Female_6Pin_2rows" H 3800 3350 50  0001 C CNN
-F 3 "http://service.powerdynamics.com/ec/Catalog17/Section%2011.pdf" H 3800 3350 50  0001 C CNN
-	1    3800 3350
+P 3950 2850
+F 0 "J2" H 3950 3217 50  0000 C CNN
+F 1 "Mini-DIN-6" H 3950 2550 50  0000 C CNN
+F 2 "Custom_Footprints:Connector_Mini-DIN_Female_6Pin_2rows" H 3950 2850 50  0001 C CNN
+F 3 "http://service.powerdynamics.com/ec/Catalog17/Section%2011.pdf" H 3950 2850 50  0001 C CNN
+	1    3950 2850
 	1    0    0    -1
 $EndComp
 $Comp
-L Connector:Jack-DC J3
+L Connector:Barrel_Jack_Switch J3
 U 1 1 5EBB033A
-P 5150 3350
-F 0 "J3" H 4920 3308 50  0000 R CNN
-F 1 "DC 12V" H 4920 3399 50  0000 R CNN
-F 2 "Connector_BarrelJack:BarrelJack_Horizontal" H 5200 3310 50  0001 C CNN
-F 3 "~" H 5200 3310 50  0001 C CNN
-	1    5150 3350
+P 5550 3350
+F 0 "J3" H 5320 3308 50  0000 R CNN
+F 1 "DC 12V" H 5320 3399 50  0000 R CNN
+F 2 "Connector_BarrelJack:BarrelJack_Horizontal" H 5600 3310 50  0001 C CNN
+F 3 "~" H 5600 3310 50  0001 C CNN
+	1    5550 3350
 	-1   0    0    1
 $EndComp
@@
 $EndComp
 Wire Wire Line
-	4100 3450 4850 3450
+	3050 3250 3200 3250
 Wire Wire Line
-	4100 3250 4850 3250
+	3050 3350 3200 3350
 Wire Wire Line
-	3300 3350 3050 3350
+	5250 3250 5150 3250
 Wire Wire Line
-	3500 3250 3050 3250
+	5250 3450 5150 3450
+Text Label 3650 2550 1    50   ~ 0
++12V
+Text Label 4250 2550 1    50   ~ 0
++12V
+Text Label 4050 2550 1    50   ~ 0
++5V
+Text Label 4150 2550 1    50   ~ 0
++5V
+Text Label 5150 3250 0    50   ~ 0
+GND
+Text Label 5150 3450 0    50   ~ 0
++12V
+Text Label 3200 3250 0    50   ~ 0
+GND
+Text Label 3200 3350 0    50   ~ 0
++5V
+Text Label 3750 2550 1    50   ~ 0
+GND
+Text Label 3450 2850 0    50   ~ 0
+GND
+Text Label 3850 2550 1    50   ~ 0
+GND
 Wire Wire Line
-	4100 3600 3300 3600
+	3750 2550 3850 2550
 Wire Wire Line
-	3300 3600 3300 3350
-Wire Wire Line
-	4100 3350 4100 3600
+	4050 2550 4150 2550
+$Comp
+L Connector:Conn_01x04_Male J4
+U 1 1 5ECBE526
+P 4100 3800
+F 0 "J4" H 4206 4078 50  0000 C CNN
+F 1 "Conn_01x04_Male" H 4206 3987 50  0000 C CNN
+F 2 "Connector_PinHeader_2.54mm:PinHeader_1x04_P2.54mm_Vertical" H 4100 3800 50  0001 C CNN
+F 3 "~" H 4100 3800 50  0001 C CNN
+	1    4100 3800
+	1    0    0    -1
+$EndComp
+Text Label 4300 3900 0    50   ~ 0
+GND
+Text Label 4300 4000 0    50   ~ 0
++5V
+Text Label 4300 3700 0    50   ~ 0
++12V
+Text Label 4300 3800 0    50   ~ 0
+SW
+Text Label 5250 3350 0    50   ~ 0
+SW
+Text Label 2000 2600 0    50   ~ 0
+GND
+Text Label 1700 3250 0    50   ~ 0
+GND
+$Comp
+L Mechanical:MountingHole_Pad H1
+U 1 1 5ECA7F49
+P 2000 2500
+F 0 "H1" H 2100 2551 50  0000 L CNN
+F 1 "MountingHole_Pad" H 2100 2460 50  0000 L CNN
+F 2 "MountingHole:MountingHole_2.2mm_M2_Pad_Via" H 2000 2500 50  0001 C CNN
+F 3 "~" H 2000 2500 50  0001 C CNN
+	1    2000 2500
+	1    0    0    -1
+$EndComp
+$Comp
+L Mechanical:MountingHole_Pad H2
+U 1 1 5ECA8016
+P 1700 3150
+F 0 "H2" H 1800 3201 50  0000 L CNN
+F 1 "MountingHole_Pad" H 1800 3110 50  0000 L CNN
+F 2 "MountingHole:MountingHole_2.2mm_M2_Pad_Via" H 1700 3150 50  0001 C CNN
+F 3 "~" H 1700 3150 50  0001 C CNN
+	1    1700 3150
+	1    0    0    -1
+$EndComp
 $EndSCHEMATC

Commit message: Swap +5V and GND
Connections:
- net +12V: no longer J2.1, J4.1 (Pin_1)
- net +5V: now also J2.6; no longer J2.3, J2.5, J4.4 (Pin_4)
- net GND: now also J2.3, J2.5, J4.4 (Pin_4); no longer J2.4, J2.6, J4.3 (Pin_3)
- net SW: now also J4.3 (Pin_3); no longer J4.2 (Pin_2)
- new net +12Vb: J2.1, J4.1 (Pin_1)
- new net +5Vb: J2.4, J4.2 (Pin_2)
Changed lines of the file:
@@
 +12V
 Text Label 4250 2550 1    50   ~ 0
-+12V
-Text Label 4050 2550 1    50   ~ 0
-+5V
-Text Label 4150 2550 1    50   ~ 0
-+5V
++12Vb
+Text Label 3750 2550 1    50   ~ 0
++5Vb
 Text Label 5150 3250 0    50   ~ 0
 GND
@@
 Text Label 3200 3350 0    50   ~ 0
 +5V
-Text Label 3750 2550 1    50   ~ 0
+Text Label 4050 2550 1    50   ~ 0
 GND
 Text Label 3450 2850 0    50   ~ 0
 GND
-Text Label 3850 2550 1    50   ~ 0
+Text Label 4150 2550 1    50   ~ 0
 GND
-Wire Wire Line
-	3750 2550 3850 2550
-Wire Wire Line
-	4050 2550 4150 2550
 $Comp
 L Connector:Conn_01x04_Male J4
@@
 	1    0    0    -1
 $EndComp
+Text Label 4300 4000 0    50   ~ 0
+GND
+Text Label 4300 3800 0    50   ~ 0
++5Vb
+Text Label 4300 3700 0    50   ~ 0
++12Vb
 Text Label 4300 3900 0    50   ~ 0
-GND
-Text Label 4300 4000 0    50   ~ 0
-+5V
-Text Label 4300 3700 0    50   ~ 0
-+12V
-Text Label 4300 3800 0    50   ~ 0
 SW
 Text Label 5250 3350 0    50   ~ 0
@@
 	1    0    0    -1
 $EndComp
+Text Label 3850 2550 1    50   ~ 0
++5V
 $EndSCHEMATC

Commit message: Add gitignore
Use github provided gitignore
Connections:
- net +12V: now also J3.2; no longer J3.1
- net GND: now also J3.1; no longer J3.2
Changed lines of the file:
@@
 Text Label 3750 2550 1    50   ~ 0
 +5Vb
+Text Label 5150 3450 0    50   ~ 0
+GND
 Text Label 5150 3250 0    50   ~ 0
-GND
-Text Label 5150 3450 0    50   ~ 0
 +12V
 Text Label 3200 3250 0    50   ~ 0
